File: Display.kicad_sch (KiCad schematic)
At the start: 23 parts, among them U10 DMG1013T-7, U11 DMG1013T-7, U12 DMG1013T-7, U13 DMG1013T-7, U14 DMG1013T-7, U15 DMG1013T-7, U16 DMG1013T-7, U17 DMG1013T-7, U26 SN74CBT3251DBQR, U65 DMG1013T-7, U66 DMG1013T-7, U8 COM-21215, U9 COM-21215

Commit message: Changed how the 14-segment displays were controlled to just use a couple shift registers
Parts:
- removed U10, U11, U12, U13, U14, U15, U16, U17, U65, U66: DMG1013T-7, Package_TO_SOT_SMD:SOT-523, symbol CMPE2750:DMG1013T-7
- removed U26: SN74CBT3251DBQR, DBQ16, symbol CMPE2750:SN74CBT3251DBQR
- removed U8, U9: COM-21215, COM-21215, symbol CMPE2750:COM-21215
- added D19, D2, D20, D21, D22, D23, D24, D25, D26, D27, D28, D29, D30, D31: NSI45015WT1G, Diode_SMD:D_SOD-123, symbol Device:D_Current-regulator
- added Q17, Q18, Q19, Q20, Q21, Q22, Q23, Q24, Q25, Q26, Q27, Q28, Q29, Q30, Q31, Q32, Q33, Q34, Q35, Q36, Q37, Q38, Q39, Q40, Q41, Q42, Q43, Q44, Q45, Q46, Q47, Q48, Q49, Q50, Q51, Q52: 2N7002K, Package_TO_SOT_SMD:SOT-23, symbol Transistor_FET:2N7002K
- added Q53, Q54, Q55, Q56, Q57, Q58, Q59, Q60, Q61, Q62, Q63, Q64, Q65, Q66: 2N7002, Package_TO_SOT_SMD:SOT-23, symbol Transistor_FET:2N7002
- added R100, R101, R102, R103, R104, R105, R106, R107, R108, R109, R110, R111, R112, R113, R114, R27, R28, R29, R30, R31, R32, R33, R34, R35, R36, R37, R38, R39, R40, R75, R76, R77, R78, R79, R80, R81, R82, R83, R84, R85, R86, R87, R88, R89, R90, R91, R92, R93, R94, R95, R96, R97, R98, R99: 4.7kΩ, Resistor_SMD:R_1206_3216Metric, symbol Device:R_US
- added U10, U11, U8, U9: SN74AHC594PWR, PW0016A_N, symbol CMPE2750:SN74AHC594PWR
- added U12, U13: COM-21215, COM-21215, symbol CMPE2750:COM-21215
Connections:
- net kathodes/top_7 is gone; now on net VBUS: R65.1
- net GND: now also Q17.2 (S), Q19.2 (S), Q21.2 (S), Q23.2 (S), Q25.2 (S), Q27.2 (S), Q29.2 (S), Q31.2 (S), Q33.2 (S), Q35.2 (S), Q37.2 (S), Q39.2 (S), Q41.2 (S), Q43.2 (S), Q45.2 (S), Q47.2 (S), Q49.2 (S), Q51.2 (S), Q53.2 (S), Q54.2 (S), Q55.2 (S), Q56.2 (S), Q57.2 (S), Q58.2 (S), Q59.2 (S), Q60.2 (S), Q61.2 (S), Q62.2 (S), Q63.2 (S), Q64.2 (S), Q65.2 (S), Q66.2 (S), R101.1, R103.1, R105.1, R107.1, R109.1, R111.1, R113.1, R88.1, R89.1, R91.1, R93.1, R95.1, R97.1, R99.1, U10.8 (GND), U11.8 (GND), U8.8 (GND), U9.8 (GND)
- net VBUS: now also R19.1, R20.1, R21.1, R22.1, R23.1, R24.1, R25.1, R26.1, R74.1, Q18.3 (D), Q20.3 (D), Q22.3 (D), Q24.3 (D), Q26.3 (D), Q28.3 (D), Q30.3 (D), Q32.3 (D), Q34.3 (D), Q36.3 (D), Q38.3 (D), Q40.3 (D), Q42.3 (D), Q44.3 (D), Q46.3 (D), Q48.3 (D), Q50.3 (D), Q52.3 (D), R27.1, R28.1, R29.1, R30.1, R31.1, R32.1, R33.1, R34.1, R35.1, R36.1, R37.1, R38.1, R39.1, R40.1, R75.1, R76.1, R77.1, R78.1, R79.1, R80.1, R81.1, R82.1, R83.1, R84.1, R85.1, R86.1
- net p16: now reaches R20.2
- net p16: now also Q17.1 (G), U9.7 (QH)
- net p31: now reaches R65.2
- net p31: now also Q39.1 (G), U11.6 (QG)
- net p2: now reaches R25.2
- net p2: now also Q23.1 (G), U8.1 (QB)
- net at R24.2: now also Q21.3 (D), Q22.1 (G)
- net at R19.2: now also Q17.3 (D), Q18.1 (G)
- net at R26.2: now also Q23.3 (D), Q24.1 (G)
- net p15: now reaches R23.2
- net p15: now also Q21.1 (G), U9.6 (QG)
- net p1: now reaches R21.2
- net p1: now also Q19.1 (G), U8.15 (QA)
- net at R22.2: now also Q19.3 (D), Q20.1 (G)
- net kathodes/bottom_7: no longer names the net of R74.2
- net kathodes/bottom_7: now also Q39.3 (D), Q40.1 (G)
- new net: D30.1 (K), Q65.3 (D)
- new net: Q41.3 (D), Q42.1 (G), R76.2
- new net: Q49.3 (D), Q50.1 (G), R84.2
- new net: Q53.1 (G), R87.2
- new net: Q51.3 (D), Q52.1 (G), R86.2
- new net: U8.9 (QH'), U9.14 (SER)
- new net: D27.1 (K), Q62.3 (D)
- new net: Q65.1 (G), R112.2
- new net: Q43.3 (D), Q44.1 (G), R78.2
- new net: Q25.3 (D), Q26.1 (G), R28.2
- new net: D24.1 (K), Q59.3 (D)
- new net: Q27.3 (D), Q28.1 (G), R30.2
- new net: Q31.3 (D), Q32.1 (G), R34.2
- new net: U10.14 (SER), U9.9 (QH')
- new net: Q45.3 (D), Q46.1 (G), R80.2
- new net: D22.1 (K), Q57.3 (D)
- new net: Q55.1 (G), R92.2
- new net: D20.1 (K), Q55.3 (D)
- new net: Q37.3 (D), Q38.1 (G), R40.2
- new net: Q62.1 (G), R106.2
- new net: Q63.1 (G), R108.2
- new net: D28.1 (K), Q63.3 (D)
- new net: Q64.1 (G), R110.2
- new net: Q66.1 (G), R114.2
- new net: D19.1 (K), Q54.3 (D)
- new net: Q29.3 (D), Q30.1 (G), R32.2
- new net: D29.1 (K), Q64.3 (D)
- new net: Q47.3 (D), Q48.1 (G), R82.2
- new net: Q61.1 (G), R104.2
- new net: Q54.1 (G), R90.2
- new net: Q56.1 (G), R94.2
- new net: D21.1 (K), Q56.3 (D)
- new net: Q35.3 (D), Q36.1 (G), R38.2
- new net: Q59.1 (G), R100.2
- new net: D2.1 (K), Q53.3 (D)
- new net: Q33.3 (D), Q34.1 (G), R36.2
- new net: D31.1 (K), Q66.3 (D)
- new net: D26.1 (K), Q61.3 (D)
- new net: Q57.1 (G), R96.2
- new net: U10.9 (QH'), U11.14 (SER)
- new net: Q58.1 (G), R98.2
- new net: D23.1 (K), Q58.3 (D)
- new net: D25.1 (K), Q60.3 (D)
- new net: Q60.1 (G), R102.2
- new net RCLK: U10.12 (RCLK), U11.12 (RCLK), U8.12 (RCLK), U9.12 (RCLK)
- new net SER: U8.14 (SER)
- new net SRCLK: U10.11 (SRCLK), U11.11 (SRCLK), U8.11 (SRCLK), U9.11 (SRCLK)
- new net VDD: U10.16 (VCC), U11.16 (VCC), U8.16 (VCC), U9.16 (VCC)
- new net b1: Q38.2 (S), U13.1
- new net b10: Q48.2 (S), U13.10
- new net b11: Q46.2 (S), U13.11
- new net b12: D30.2 (A)
- new net b13: D26.2 (A), U13.13
- new net b14: D25.2 (A), U13.14
- new net b15: Q40.2 (S), U13.15
- new net b16: Q36.2 (S), U13.16
- new net b2: Q42.2 (S), U13.2
- new net b3: D28.2 (A)
- new net b4: D27.2 (A), U13.4
- new net b5: D31.2 (A), U13.3
- new net b6: D29.2 (A), U13.6
- new net b7: Q44.2 (S), U13.12, U13.7
- new net b8: Q50.2 (S), U13.5, U13.8
- new net b9: Q52.2 (S), U13.9
- new net p10: Q29.1 (G), R31.2, U9.1 (QB)
- new net p11: Q27.1 (G), R29.2, U9.2 (QC)
- new net p12: R97.2, R98.1, U9.3 (QD)
- new net p13: R89.2, R90.1, U9.4 (QE)
- new net p14: R87.1, R88.2, U9.5 (QF)
- new net p17: Q37.1 (G), R39.2, U10.15 (QA)
- new net p18: Q41.1 (G), R75.2, U10.1 (QB)
- new net p19: R107.2, R108.1, U10.2 (QC)
- new net p20: R105.2, R106.1, U10.3 (QD)
- new net p21: R113.2, R114.1, U10.4 (QE)
- new net p22: R109.2, R110.1, U10.5 (QF)
- new net p23: Q43.1 (G), R77.2, U10.6 (QG)
- new net p24: Q49.1 (G), R83.2, U10.7 (QH)
- new net p25: Q51.1 (G), R85.2, U11.15 (QA)
- new net p26: Q47.1 (G), R81.2, U11.1 (QB)
- new net p27: Q45.1 (G), R79.2, U11.2 (QC)
- new net p28: R111.2, R112.1, U11.3 (QD)
- new net p29: R103.2, R104.1, U11.4 (QE)
- new net p3: R93.2, R94.1, U8.2 (QC)
- new net p30: R101.2, R102.1, U11.5 (QF)
- new net p32: Q35.1 (G), R37.2, U11.7 (QH)
- new net p4: R91.2, R92.1, U8.3 (QD)
- new net p5: R100.1, R99.2, U8.4 (QE)
- new net p6: R95.2, R96.1, U8.5 (QF)
- new net p7: Q25.1 (G), R27.2, U8.6 (QG)
- new net p8: Q31.1 (G), R33.2, U8.7 (QH)
- new net p9: Q33.1 (G), R35.2, U9.15 (QA)
- new net t1: Q20.2 (S), U12.1
- new net t10: Q30.2 (S), U12.10
- new net t11: Q28.2 (S), U12.11
- new net t12: D23.2 (A)
- new net t13: D19.2 (A), U12.13
- new net t14: D2.2 (A), U12.14
- new net t15: Q22.2 (S), U12.15
- new net t16: Q18.2 (S), U12.16
- new net t2: Q24.2 (S), U12.2
- new net t3: D21.2 (A)
- new net t4: D20.2 (A), U12.4
- new net t5: D24.2 (A), U12.3
- new net t6: D22.2 (A), U12.6
- new net t7: Q26.2 (S), U12.12, U12.7
- new net t8: Q32.2 (S), U12.5, U12.8
- new net t9: Q34.2 (S), U12.9
- new net ~{RCL}: U10.13 (RCLR_N), U11.13 (RCLR_N), U8.13 (RCLR_N), U9.13 (RCLR_N)
- new net ~{SRCLR}: U10.10 (SRCLR_N), U11.10 (SRCLR_N), U8.10 (SRCLR_N), U9.10 (SRCLR_N)
- no-connect marks 0 -> 1
Other:
- removed sheet current
- removed sheet kathodes

Commit message: Finished the display and input switch schematics. Also added input buffers to the inputs and made them differential
Parts:
- added R115, R116, R117, R118, R119, R120, R121, R122, R123, R124, R125, R126, R127, R128, R129, R130, R131, R132: 4.7kΩ, Resistor_SMD:R_1206_3216Metric, symbol Device:R_US
Connections:
- net VBUS: now also R117.1, R118.1, R120.1, R121.1, R123.1, R124.1, R126.1, R127.1, R129.1, R130.1, R132.1; no longer R22.1, R25.1, R28.1, R31.1, R34.1, R38.1, R65.1, R76.1, R79.1, R82.1, R85.1
- net p1: now also R22.1; no longer Q19.1 (G)
- net p10: now also R36.2, R116.1; no longer Q29.1 (G), R31.2
- net p11: now also R33.2, R34.1; no longer Q27.1 (G), R29.2
- net p15: now also R24.2, R25.1; no longer Q21.1 (G), R23.2
- net p16: now also R115.1; no longer Q17.1 (G)
- net p17: now also R40.2, R65.1; no longer Q37.1 (G), R39.2
- net p18: now also R78.2, R79.1; no longer Q41.1 (G), R75.2
- net p2: now also R27.2, R28.1; no longer Q23.1 (G), R25.2
- net p23: now also R81.2, R82.1; no longer Q43.1 (G), R77.2
- net p24: now also R127.2, R128.1; no longer Q49.1 (G), R83.2
- net p25: now also R130.2, R131.1; no longer Q51.1 (G), R85.2
- net p26: now also R124.2, R125.1; no longer Q47.1 (G), R81.2
- net p27: now also R84.2, R85.1; no longer Q45.1 (G), R79.2
- net p31: now also R75.2, R76.1; no longer Q39.1 (G), R65.2
- net p32: now also R38.1; no longer Q35.1 (G)
- net p7: now also R30.2, R31.1; no longer Q25.1 (G), R27.2
- net p8: now also R118.2, R119.1; no longer Q31.1 (G), R33.2
- net p9: now also R121.2, R122.1; no longer Q33.1 (G), R35.2
- net at Q41.3 (D), Q42.1 (G): now also R80.2; no longer R76.2
- net at Q49.3 (D), Q50.1 (G): now also R129.2; no longer R84.2
- net at Q51.3 (D), Q52.1 (G): now also R132.2; no longer R86.2
- net at Q19.3 (D), Q20.1 (G): now also R23.2; no longer R22.2
- net at Q43.3 (D), Q44.1 (G): now also R83.2; no longer R78.2
- net at Q25.3 (D), Q26.1 (G): now also R32.2; no longer R28.2
- net at Q27.3 (D), Q28.1 (G): now also R35.2; no longer R30.2
- net at Q23.3 (D), Q24.1 (G): now also R29.2; no longer R26.2
- net at Q39.3 (D), Q40.1 (G): now also R77.2; no longer R74.2
- net at Q31.3 (D), Q32.1 (G): now also R120.2; no longer R34.2
- net at Q45.3 (D), Q46.1 (G): now also R86.2; no longer R80.2
- net at Q37.3 (D), Q38.1 (G): now also R74.2; no longer R40.2
- net at Q29.3 (D), Q30.1 (G): now also R117.2; no longer R32.2
- net at Q47.3 (D), Q48.1 (G): now also R126.2; no longer R82.2
- net at Q35.3 (D), Q36.1 (G): now also R39.2; no longer R38.2
- net at Q33.3 (D), Q34.1 (G): now also R123.2; no longer R36.2
- net at Q21.3 (D), Q22.1 (G): now also R26.2; no longer R24.2
- new net: Q27.1 (G), R34.2
- new net: Q41.1 (G), R79.2
- new net: Q37.1 (G), R65.2
- new net: Q25.1 (G), R31.2
- new net: Q21.1 (G), R25.2
- new net: Q35.1 (G), R38.2
- new net: Q17.1 (G), R115.2
- new net: Q45.1 (G), R85.2
- new net: Q23.1 (G), R28.2
- new net: Q49.1 (G), R128.2
- new net: Q47.1 (G), R125.2
- new net: Q33.1 (G), R122.2
- new net: Q51.1 (G), R131.2
- new net: Q31.1 (G), R119.2
- new net: Q29.1 (G), R116.2
- new net: Q43.1 (G), R82.2
- new net: Q19.1 (G), R22.2
- new net: Q39.1 (G), R76.2
Other:
- moved on the sheet: R20

Commit message: Almost done. Just going to try and change something
Parts:
- added C18, C19, C20, C21: 100nF, LMK212G_TAY, symbol CMPE2750:LMK212B7105KGHTR
- added J9: Conn_01x02, symbol Connector_Generic:Conn_01x02
Connections:
- net VBUS: now also J9.1 (Pin_1); no longer Q18.3 (D), Q20.3 (D), Q22.3 (D), Q24.3 (D), Q26.3 (D), Q28.3 (D), Q30.3 (D), Q32.3 (D), Q34.3 (D), Q36.3 (D), Q38.3 (D), Q40.3 (D), Q42.3 (D), Q44.3 (D), Q46.3 (D), Q48.3 (D), Q50.3 (D), Q52.3 (D), R117.1, R118.1, R120.1, R121.1, R123.1, R124.1, R126.1, R127.1, R129.1, R130.1, R132.1, R19.1, R20.1, R21.1, R23.1, R24.1, R26.1, R27.1, R29.1, R30.1, R32.1, R33.1, R35.1, R36.1, R37.1, R39.1, R40.1, R74.1, R75.1, R77.1, R78.1, R80.1, R81.1, R83.1, R84.1, R86.1
- net VDD: now also C18.1, C19.1, C20.1, C21.1
- net SO: now reaches U11.9 (QH')
- new net -5V: C18.2, C19.2, C20.2, C21.2
- new net V_{DISP}: J9.2 (Pin_2), Q18.3 (D), Q20.3 (D), Q22.3 (D), Q24.3 (D), Q26.3 (D), Q28.3 (D), Q30.3 (D), Q32.3 (D), Q34.3 (D), Q36.3 (D), Q38.3 (D), Q40.3 (D), Q42.3 (D), Q44.3 (D), Q46.3 (D), Q48.3 (D), Q50.3 (D), Q52.3 (D), R117.1, R118.1, R120.1, R121.1, R123.1, R124.1, R126.1, R127.1, R129.1, R130.1, R132.1, R19.1, R20.1, R21.1, R23.1, R24.1, R26.1, R27.1, R29.1, R30.1, R32.1, R33.1, R35.1, R36.1, R37.1, R39.1, R40.1, R74.1, R75.1, R77.1, R78.1, R80.1, R81.1, R83.1, R84.1, R86.1
- no-connect marks 1 -> 0

Commit message: Schematic is done?
Parts:
- removed Q18, Q20, Q22, Q24, Q26, Q28, Q30, Q32, Q34, Q36, Q38, Q40, Q42, Q44, Q46, Q48, Q50, Q52: 2N7002K, Package_TO_SOT_SMD:SOT-23, symbol Transistor_FET:2N7002K
- added Q18, Q20, Q22, Q24, Q26, Q28, Q30, Q32, Q34, Q36, Q38, Q40, Q42, Q44, Q46, Q48, Q50, Q52: IRLML6402TRPBF, Package_TO_SOT_SMD:SOT-23, symbol Transistor_FET:IRLML6402
- C18, C19, C20, C21: footprint LMK212G_TAY -> Capacitor_SMD:C_0402_1005Metric; symbol CMPE2750:LMK212B7105KGHTR -> CMPE2750:CL05B104KP5NNNC
- J9: footprint (none) -> Connector_PinHeader_2.54mm:PinHeader_1x02_P2.54mm_Vertical
- Q17, Q19, Q21, Q23, Q25, Q27, Q29, Q31, Q33, Q35, Q37, Q39, Q41, Q43, Q45, Q47, Q49, Q51: value 2N7002K -> 2N7002; symbol Transistor_FET:2N7002K -> Transistor_FET:2N7002
- U10, U11, U8, U9: footprint PW0016A_N -> Package_SO:TSSOP-16_4.4x5mm_P0.65mm
Connections:
- net GND: now also R118.1, R121.1, R124.1, R127.1, R130.1, R20.1, R21.1, R24.1, R27.1, R30.1, R33.1, R36.1, R37.1, R40.1, R75.1, R78.1, R81.1, R84.1
- net V_{DISP}: now also Q18.2 (S), Q20.2 (S), Q22.2 (S), Q24.2 (S), Q26.2 (S), Q28.2 (S), Q30.2 (S), Q32.2 (S), Q34.2 (S), Q36.2 (S), Q38.2 (S), Q40.2 (S), Q42.2 (S), Q44.2 (S), Q46.2 (S), Q48.2 (S), Q50.2 (S), Q52.2 (S); no longer R118.1, R121.1, R124.1, R127.1, R130.1, R20.1, R21.1, R24.1, R27.1, R30.1, R33.1, R36.1, R37.1, R40.1, R75.1, R78.1, R81.1, R84.1
- net b1: now also Q38.3 (D)
- net b10: now also Q48.3 (D)
- net b11: now also Q46.3 (D)
- net b15: now also Q40.3 (D)
- net b16: now also Q36.3 (D)
- net b2: now also Q42.3 (D)
- net b7: now also Q44.3 (D)
- net b8: now also Q50.3 (D)
- net b9: now also Q52.3 (D)
- net t1: now also Q20.3 (D)
- net t10: now also Q30.3 (D)
- net t11: now also Q28.3 (D)
- net t15: now also Q22.3 (D)
- net t16: now also Q18.3 (D)
- net t2: now also Q24.3 (D)
- net t7: now also Q26.3 (D)
- net t8: now also Q32.3 (D)
- net t9: now also Q34.3 (D)
- net at Q27.3 (D), R35.2: now also Q28.1 (G)
- net at Q37.3 (D), R74.2: now also Q38.1 (G)
- net at Q33.3 (D), R123.2: now also Q34.1 (G)
- net at Q29.3 (D), R117.2: now also Q30.1 (G)
- net at Q41.3 (D), R80.2: now also Q42.1 (G)
- net at Q17.3 (D), R19.2: now also Q18.1 (G)
- net at Q21.3 (D), R26.2: now also Q22.1 (G)
- net at Q49.3 (D), R129.2: now also Q50.1 (G)
- net at Q25.3 (D), R32.2: now also Q26.1 (G)
- net at Q19.3 (D), R23.2: now also Q20.1 (G)
- net at Q47.3 (D), R126.2: now also Q48.1 (G)
- net at Q31.3 (D), R120.2: now also Q32.1 (G)
- net at Q51.3 (D), R132.2: now also Q52.1 (G)
- net at Q35.3 (D), R39.2: now also Q36.1 (G)
- net at Q45.3 (D), R86.2: now also Q46.1 (G)
- net at Q39.3 (D), R77.2: now also Q40.1 (G)
- net at Q43.3 (D), R83.2: now also Q44.1 (G)
- net at Q23.3 (D), R29.2: now also Q24.1 (G)
Other:
- note added: "(these were originally pull-up resistors and I'm too tired to make them all go downward)"

Commit message: *Now* it's finished. Maybe.
Parts:
- added C31: 10µF, Capacitor_SMD:C_1206_3216Metric, symbol CMPE2750:CL31A106KOHNNNE
Connections:
- net GND: now also C31.2
- net V_{DISP}: now also C31.1
Changed lines of the file:
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@@
 	(wire
 		(pts
+			(xy 458.47 157.48) (xy 458.47 156.21)
+		)
+		(stroke
+			(width 0)
+			(type default)
+		)
+	)
+	(wire
+		(pts
 			(xy 331.47 80.01) (xy 331.47 82.55)
 		)
@@
 	(wire
 		(pts
+			(xy 458.47 147.32) (xy 458.47 148.59)
+		)
+		(stroke
+			(width 0)
+			(type default)
+		)
+	)
+	(wire
+		(pts
 			(xy 176.53 87.63) (xy 176.53 80.01)
 		)
@@
 		)
 	)
+	(label "V_{DISP}"
+		(at 458.47 147.32 180)
+		(fields_autoplaced yes)
+		(effects
+			(font
+				(size 1.27 1.27)
+			)
+			(justify right bottom)
+		)
+	)
 	(label "p28"
 		(at 342.9 207.01 180)
@@
 	)
 	(symbol
+		(lib_id "CMPE2750:CL31A106KOHNNNE")
+		(at 458.47 148.59 270)
+		(unit 1)
+		(exclude_from_sim no)
+		(in_bom yes)
+		(on_board yes)
+		(dnp no)
+		(fields_autoplaced yes)
+		(property "Reference" "C31"
+			(at 462.28 151.1299 90)
+			(effects
+				(font
+					(size 1.524 1.524)
+				)
+				(justify left)
+			)
+		)
+		(property "Value" "10µF"
+			(at 462.28 153.6699 90)
+			(effects
+				(font
+					(size 1.524 1.524)
+				)
+				(justify left)
+			)
+		)
+		(property "Footprint" "Capacitor_SMD:C_1206_3216Metric"
+			(at 458.47 148.59 0)
+			(effects
+				(font
+					(size 1.27 1.27)
+					(italic yes)
+				)
+				(hide yes)
+			)
+		)
+		(property "Datasheet" "CL31A106KOHNNNE"
+			(at 458.47 148.59 0)
+			(effects
+				(font
+					(size 1.27 1.27)
+					(italic yes)
+				)
+				(hide yes)
+			)
+		)
+		(property "Description" ""
+			(at 458.47 148.59 0)
+			(effects
+				(font
+					(size 1.27 1.27)
+				)
+				(hide yes)
+			)
+		)
+		(pin "2"
+		)
+		(pin "1"
+		)
+		(instances
+			(project ""
+				(path "/a86318a1-888d-4137-89a5-221e5a1bc171/d57d4e03-f6b9-4171-ade1-ebcfed743b5a"
+					(reference "C31")
+					(unit 1)
+				)
+			)
+		)
+	)
+	(symbol
 		(lib_id "Device:R_US")
 		(at 439.42 40.64 0)
@@
 					(unit 1)
 				)
+			)
+		)
+	)
+	(symbol
+		(lib_id "power:GND")
+		(at 458.47 157.48 0)
+		(unit 1)
+		(exclude_from_sim no)
+		(in_bom yes)
+		(on_board yes)
+		(dnp no)
+		(fields_autoplaced yes)
+		(property "Reference" "#PWR0165"
+			(at 458.47 163.83 0)
+			(effects
+				(font
+					(size 1.27 1.27)
+				)
+				(hide yes)
+			)
+		)
+		(property "Value" "GND"
+			(at 458.47 162.56 0)
+			(effects
+				(font
+					(size 1.27 1.27)
+				)
+			)
+		)
+		(property "Footprint" ""
+			(at 458.47 157.48 0)
+			(effects
+				(font
+					(size 1.27 1.27)
+				)
+				(hide yes)
+			)
+		)
+		(property "Datasheet" ""
+			(at 458.47 157.48 0)
+			(effects
+				(font
+					(size 1.27 1.27)
+				)
+				(hide yes)
+			)
+		)
+		(property "Description" "Power symbol creates a global label with name \"GND\" , ground"
+			(at 458.47 157.48 0)
+			(effects
+				(font
+					(size 1.27 1.27)
+				)
+				(hide yes)
+			)
+		)
+		(pin "1"
+		)
+		(instances
+			(project ""
+				(path "/a86318a1-888d-4137-89a5-221e5a1bc171/d57d4e03-f6b9-4171-ade1-ebcfed743b5a"
+					(reference "#PWR0165")
+					(unit 1)
+				)

Commit message: Swapped the current limiting diodes for resistors. They *should* be good enough under normal operating conditions. Also added some pull-down resistors. Done?
Parts:
- removed D19, D2, D20, D21, D22, D23, D24, D25, D26, D27, D28, D29, D30, D31: NSI45015WT1G, Diode_SMD:D_SOD-123, symbol Device:D_Current-regulator
- added R161, R162, R163, R164, R165, R166, R167, R168, R169, R170, R171, R172, R173, R174: 133Ω, Resistor_SMD:R_0603_1608Metric, symbol CMPE2750:RT0603BRD07133RL
Connections:
- net b12: now also R173.1
- net b13: now also R169.1
- net b14: now also R168.1
- net b3: now also R171.1
- net b4: now also R170.1
- net b5: now also R174.1
- net b6: now also R172.1
- net t12: now also R166.1
- net t13: now also R162.1
- net t14: now also R161.1
- net t3: now also R164.1
- net t4: now also R163.1
- net t5: now also R167.1
- net t6: now also R165.1
- net at Q65.3 (D): now also R173.2
- net at Q62.3 (D): now also R170.2
- net at Q59.3 (D): now also R167.2
- net at Q57.3 (D): now also R165.2
- net at Q55.3 (D): now also R163.2
- net at Q63.3 (D): now also R171.2
- net at Q54.3 (D): now also R162.2
- net at Q64.3 (D): now also R172.2
- net at Q56.3 (D): now also R164.2
- net at Q53.3 (D): now also R161.2
- net at Q66.3 (D): now also R174.2
- net at Q61.3 (D): now also R169.2
- net at Q58.3 (D): now also R166.2
- net at Q60.3 (D): now also R168.2

Commit message: Added mounting holes to the schematic, reset the annotations, updated a few footprints, and fixed some issues that were discovered on the ERC.
Parts:
- U10: renamed from U12; footprint COM-21215 -> CMPE2750:COM-21215
- U11: renamed from U13; footprint COM-21215 -> CMPE2750:COM-21215
- renumbered C18 to C25, C19 to C26, C31 to C27, C20 to C28, C21 to C29, Q18 to Q1, Q17 to Q10, Q19 to Q11, Q21 to Q12, Q23 to Q13, Q25 to Q14, Q27 to Q15, Q29 to Q16, Q31 to Q17, Q33 to Q18, Q36 to Q19, Q20 to Q2, Q38 to Q20, Q40 to Q21, Q42 to Q22, Q44 to Q23, Q46 to Q24, Q48 to Q25, Q50 to Q26, Q52 to Q27, Q35 to Q28, Q37 to Q29, Q22 to Q3, Q39 to Q30, Q41 to Q31, Q43 to Q32, Q45 to Q33, Q47 to Q34, Q49 to Q35, Q51 to Q36, Q58 to Q37, Q53 to Q38, Q54 to Q39, Q24 to Q4, Q55 to Q40, Q56 to Q41, Q57 to Q42, Q59 to Q43, Q65 to Q44, Q60 to Q45, Q61 to Q46, Q62 to Q47, Q63 to Q48, Q64 to Q49, Q26 to Q5, Q66 to Q50, Q28 to Q6, Q30 to Q7, Q32 to Q8, Q34 to Q9, R131 to R100, R166 to R101, R161 to R102, R162 to R103, R163 to R104, R164 to R105, R165 to R106, R167 to R107, R98 to R108, R87 to R109, R90 to R110, R92 to R111, R94 to R112, R96 to R113, R100 to R114, R97 to R115, R88 to R116, R89 to R117, R91 to R118, R93 to R119, R95 to R120, R99 to R121, R173 to R122, R171 to R123, R172 to R124, R168 to R125, R170 to R126, R174 to R127, R169 to R128, R112 to R129, R102 to R130, R104 to R131, R106 to R132, R108 to R133, R110 to R134, R114 to R135, R111 to R136, R101 to R137, R103 to R138, R105 to R139, R107 to R140, R109 to R141, R113 to R142, R19 to R47, R23 to R48, R26 to R49, R29 to R50, R32 to R51, R35 to R52, R117 to R53, R120 to R54, R123 to R55, R20 to R56, R21 to R57, R24 to R58, R27 to R59, R30 to R60, R33 to R61, R36 to R62, R118 to R63, R121 to R64, R115 to R65, R22 to R66, R25 to R67, R28 to R68, R31 to R69, R34 to R70, R116 to R71, R119 to R72, R122 to R73, R39 to R74, R74 to R75, R77 to R76, R80 to R77, R83 to R78, R86 to R79, R126 to R80, R129 to R81, R132 to R82, R37 to R83, R40 to R84, R75 to R85, R78 to R86, R81 to R87, R84 to R88, R124 to R89, R127 to R90, R130 to R91, R38 to R92, R65 to R93, R76 to R94, R79 to R95, R82 to R96, R85 to R97, R125 to R98, R128 to R99, U11 to U12, U8 to U7, U9 to U8, U10 to U9
Connections:
- net b12: now also U11.12
- net b3: now also U11.3
- net b5: now also U11.5; no longer U11.3
- net b7: no longer U11.12
- net b8: no longer U11.5
- net t12: now also U10.12
- net t3: now also U10.3
- net t5: now also U10.5; no longer U10.3
- net t7: no longer U10.12
- net t8: no longer U10.5

Commit message: Added a ferrite bead and removed a decoupling cap from another ferrite bead
Parts:
- renumbered C25 to C24, C26 to C25, C27 to C26, C28 to C27, C29 to C28
