File: Display.kicad_sch (KiCad schematic)
At the start: 158 parts, among them J9 Conn_01x02, Q1 IRLML6402TRPBF, Q10 2N7002, Q11 2N7002, Q12 2N7002, Q13 2N7002, Q14 2N7002, Q15 2N7002, Q16 2N7002, Q17 2N7002, Q18 2N7002, Q19 IRLML6402TRPBF, Q2 IRLML6402TRPBF, Q20 IRLML6402TRPBF, Q21 IRLML6402TRPBF, Q22 IRLML6402TRPBF, Q23 IRLML6402TRPBF, Q24 IRLML6402TRPBF, Q25 IRLML6402TRPBF, Q26 IRLML6402TRPBF, Q27 IRLML6402TRPBF, Q28 2N7002, Q29 2N7002, Q3 IRLML6402TRPBF, Q30 2N7002, Q31 2N7002, Q32 2N7002, Q33 2N7002, Q34 2N7002, Q35 2N7002, Q36 2N7002, Q37 2N7002, Q38 2N7002, Q39 2N7002, Q4 IRLML6402TRPBF, Q40 2N7002, Q41 2N7002, Q42 2N7002, Q43 2N7002, Q44 2N7002, Q45 2N7002, Q46 2N7002, Q47 2N7002, Q48 2N7002, Q49 2N7002, Q5 IRLML6402TRPBF, Q50 2N7002, Q6 IRLML6402TRPBF, Q7 IRLML6402TRPBF, Q8 IRLML6402TRPBF, Q9 IRLML6402TRPBF, U10 COM-21215, U11 COM-21215, U12 SN74AHC594PWR, U7 SN74AHC594PWR, U8 SN74AHC594PWR, U9 SN74AHC594PWR

Commit message: Component placing partly done. Saving before overwriting the pcb with the templating script output
Parts:
- R100, R108, R109, R110, R111, R112, R113, R114, R115, R116, R117, R118, R119, R120, R121, R129, R130, R131, R132, R133, R134, R135, R136, R137, R138, R139, R140, R141, R142, R47, R48, R49, R50, R51, R52, R53, R54, R55, R56, R57, R58, R59, R60, R61, R62, R63, R64, R65, R66, R67, R68, R69, R70, R71, R72, R73, R74, R75, R76, R77, R78, R79, R80, R81, R82, R83, R84, R85, R86, R87, R88, R89, R90, R91, R92, R93, R94, R95, R96, R97, R98, R99: footprint Resistor_SMD:R_1206_3216Metric -> Resistor_SMD:R_0402_1005Metric; symbol Device:R_US -> CMPE2750:AC0402FR-074K7L
Connections:
- net -5V is gone; now on net GND: C24.2, C25.2, C27.2, C28.2
