File: filters_and_amps.kicad_sch (KiCad schematic)
At the start: 32 parts, among them J7 Conn_02x02_Counter_Clockwise, J8 Conn_02x02_Counter_Clockwise, U4 OPA1678IDR, U5 OPA1678IDR, U6 OPA1678IDR

Commit message: Added a ferrite bead and removed a decoupling cap from another ferrite bead
Parts:
- renumbered C14 to C13, C15 to C14, C16 to C15, C17 to C16, C18 to C17, C19 to C18, C20 to C19, C21 to C20, C22 to C21, C23 to C22, C24 to C23
Changed lines of the file:
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@@
 		(dnp no)
 		(fields_autoplaced yes)
-		(property "Reference" "C18"
+		(property "Reference" "C17"
 			(at 220.9863 102.87 90)
 			(effects
@@
 			(project "CMPE2750"
 				(path "/a86318a1-888d-4137-89a5-221e5a1bc171/d68b35fd-c62c-4cb2-9479-1cd357042dd9"
-					(reference "C18")
+					(reference "C17")
 					(unit 1)
 				)
@@
 		(dnp no)
 		(fields_autoplaced yes)
-		(property "Reference" "#PWR064"
+		(property "Reference" "#PWR063"
 			(at 121.92 143.51 0)
 			(effects
@@
 			(project "CMPE2750"
 				(path "/a86318a1-888d-4137-89a5-221e5a1bc171/d68b35fd-c62c-4cb2-9479-1cd357042dd9"
-					(reference "#PWR064")
+					(reference "#PWR063")
 					(unit 1)
 				)
@@
 		(dnp no)
 		(fields_autoplaced yes)
-		(property "Reference" "#PWR058"
+		(property "Reference" "#PWR057"
 			(at 179.07 60.96 0)
 			(effects
@@
 			(project "CMPE2750"
 				(path "/a86318a1-888d-4137-89a5-221e5a1bc171/d68b35fd-c62c-4cb2-9479-1cd357042dd9"
-					(reference "#PWR058")
+					(reference "#PWR057")
 					(unit 1)
 				)
@@
 		(dnp no)
 		(fields_autoplaced yes)
-		(property "Reference" "C20"
+		(property "Reference" "C19"
 			(at 46.9963 109.22 90)
 			(effects
@@
 			(project ""
 				(path "/a86318a1-888d-4137-89a5-221e5a1bc171/d68b35fd-c62c-4cb2-9479-1cd357042dd9"
-					(reference "C20")
+					(reference "C19")
 					(unit 1)
 				)
@@
 		(dnp no)
 		(fields_autoplaced yes)
-		(property "Reference" "#PWR059"
+		(property "Reference" "#PWR058"
 			(at 234.95 82.55 0)
 			(effects
@@
 			(project "CMPE2750"
 				(path "/a86318a1-888d-4137-89a5-221e5a1bc171/d68b35fd-c62c-4cb2-9479-1cd357042dd9"
-					(reference "#PWR059")
+					(reference "#PWR058")
 					(unit 1)
 				)
@@
 		(dnp no)
 		(fields_autoplaced yes)
-		(property "Reference" "C16"
+		(property "Reference" "C15"
 			(at 180.34 54.61 0)
 			(effects
@@
 			(project "CMPE2750"
 				(path "/a86318a1-888d-4137-89a5-221e5a1bc171/d68b35fd-c62c-4cb2-9479-1cd357042dd9"
-					(reference "C16")
+					(reference "C15")
 					(unit 1)
 				)
@@
 		(dnp no)
 		(fields_autoplaced yes)
-		(property "Reference" "#PWR056"
+		(property "Reference" "#PWR055"
 			(at 152.4 41.91 0)
 			(effects
@@
 			(project "CMPE2750"
 				(path "/a86318a1-888d-4137-89a5-221e5a1bc171/d68b35fd-c62c-4cb2-9479-1cd357042dd9"
-					(reference "#PWR056")
+					(reference "#PWR055")
 					(unit 1)
 				)
@@
 		(dnp no)
 		(fields_autoplaced yes)
-		(property "Reference" "C22"
+		(property "Reference" "C21"
 			(at 191.77 129.5399 90)
 			(effects
@@
 			(project "CMPE2750"
 				(path "/a86318a1-888d-4137-89a5-221e5a1bc171/d68b35fd-c62c-4cb2-9479-1cd357042dd9"
-					(reference "C22")
+					(reference "C21")
 					(unit 1)
 				)
@@
 		(dnp no)
 		(fields_autoplaced yes)
-		(property "Reference" "C23"
+		(property "Reference" "C22"
 			(at 125.73 130.8099 90)
 			(effects
@@
 			(project ""
 				(path "/a86318a1-888d-4137-89a5-221e5a1bc171/d68b35fd-c62c-4cb2-9479-1cd357042dd9"
-					(reference "C23")
+					(reference "C22")
 					(unit 1)
 				)
@@
 		(dnp no)
 		(fields_autoplaced yes)
-		(property "Reference" "#PWR051"
+		(property "Reference" "#PWR050"
 			(at 130.81 26.67 0)
 			(effects
@@
 			(project "CMPE2750"
 				(path "/a86318a1-888d-4137-89a5-221e5a1bc171/d68b35fd-c62c-4cb2-9479-1cd357042dd9"
-					(reference "#PWR051")
+					(reference "#PWR050")
 					(unit 1)
 				)
@@
 		(dnp no)
 		(fields_autoplaced yes)
-		(property "Reference" "C15"
+		(property "Reference" "C14"
 			(at 278.13 21.59 0)
 			(effects
@@
 			(project "CMPE2750"
 				(path "/a86318a1-888d-4137-89a5-221e5a1bc171/d68b35fd-c62c-4cb2-9479-1cd357042dd9"
-					(reference "C15")
+					(reference "C14")
 					(unit 1)
 				)
@@
 		(dnp no)
 		(fields_autoplaced yes)
-		(property "Reference" "#PWR052"
+		(property "Reference" "#PWR051"
 			(at 142.24 21.59 0)
 			(effects
@@
 			(project "CMPE2750"
 				(path "/a86318a1-888d-4137-89a5-221e5a1bc171/d68b35fd-c62c-4cb2-9479-1cd357042dd9"
-					(reference "#PWR052")
+					(reference "#PWR051")
 					(unit 1)
 				)
@@
 		(on_board yes)
 		(dnp no)
-		(property "Reference" "#PWR055"
+		(property "Reference" "#PWR054"
 			(at 13.97 39.37 0)
 			(effects
@@
 			(project "CMPE2750"
 				(path "/a86318a1-888d-4137-89a5-221e5a1bc171/d68b35fd-c62c-4cb2-9479-1cd357042dd9"
-					(reference "#PWR055")
+					(reference "#PWR054")
 					(unit 1)
 				)
@@
 		(dnp no)
 		(fields_autoplaced yes)
-		(property "Reference" "#PWR062"
+		(property "Reference" "#PWR061"
 			(at 236.22 139.7 0)
 			(effects
@@
 			(project "CMPE2750"
 				(path "/a86318a1-888d-4137-89a5-221e5a1bc171/d68b35fd-c62c-4cb2-9479-1cd357042dd9"
-					(reference "#PWR062")
+					(reference "#PWR061")
 					(unit 1)
 				)
@@
 		(dnp no)
 		(fields_autoplaced yes)
-		(property "Reference" "#PWR061"
+		(property "Reference" "#PWR060"
 			(at 233.68 95.25 0)
 			(effects
@@
 			(project ""
 				(path "/a86318a1-888d-4137-89a5-221e5a1bc171/d68b35fd-c62c-4cb2-9479-1cd357042dd9"
-					(reference "#PWR061")
+					(reference "#PWR060")
 					(unit 1)
 				)
@@
 		(dnp no)
 		(fields_autoplaced yes)
-		(property "Reference" "#PWR054"
+		(property "Reference" "#PWR053"
 			(at 281.94 24.13 0)
 			(effects
@@
 			(project "CMPE2750"
 				(path "/a86318a1-888d-4137-89a5-221e5a1bc171/d68b35fd-c62c-4cb2-9479-1cd357042dd9"
-					(reference "#PWR054")
+					(reference "#PWR053")
 					(unit 1)
 				)
@@
 		(dnp no)
 		(fields_autoplaced yes)
-		(property "Reference" "C24"
+		(property "Reference" "C23"
 			(at 62.23 135.8899 90)
 			(effects
@@
 			(project ""
 				(path "/a86318a1-888d-4137-89a5-221e5a1bc171/d68b35fd-c62c-4cb2-9479-1cd357042dd9"
-					(reference "C24")
+					(reference "C23")
 					(unit 1)
 				)
@@
 		(dnp no)
 		(fields_autoplaced yes)
-		(property "Reference" "#PWR057"
+		(property "Reference" "#PWR056"
 			(at 186.69 63.5 0)
 			(effects
@@
 			(project ""
 				(path "/a86318a1-888d-4137-89a5-221e5a1bc171/d68b35fd-c62c-4cb2-9479-1cd357042dd9"
-					(reference "#PWR057")
+					(reference "#PWR056")
 					(unit 1)
 				)
@@
 		(dnp no)
 		(fields_autoplaced yes)
-		(property "Reference" "C21"
+		(property "Reference" "C20"
 			(at 240.03 126.9999 90)
 			(effects
@@
 			(project "CMPE2750"
 				(path "/a86318a1-888d-4137-89a5-221e5a1bc171/d68b35fd-c62c-4cb2-9479-1cd357042dd9"
-					(reference "C21")
+					(reference "C20")
 					(unit 1)
 				)
@@
 		(dnp no)
 		(fields_autoplaced yes)
-		(property "Reference" "C19"
+		(property "Reference" "C18"
 			(at 106.6863 106.68 90)
 			(effects
@@
 			(project ""
 				(path "/a86318a1-888d-4137-89a5-221e5a1bc171/d68b35fd-c62c-4cb2-9479-1cd357042dd9"
-					(reference "C19")
+					(reference "C18")
 					(unit 1)
 				)
@@
 		(dnp no)
 		(fields_autoplaced yes)
-		(property "Reference" "C17"
+		(property "Reference" "C16"
 			(at 176.5363 102.87 90)
 			(effects
@@
 			(project "CMPE2750"
 				(path "/a86318a1-888d-4137-89a5-221e5a1bc171/d68b35fd-c62c-4cb2-9479-1cd357042dd9"
-					(reference "C17")
+					(reference "C16")
 					(unit 1)
 				)
@@
 		(dnp no)
 		(fields_autoplaced yes)
-		(property "Reference" "C14"
+		(property "Reference" "C13"
 			(at 138.43 19.05 0)
 			(effects
@@
 			(project "CMPE2750"
 				(path "/a86318a1-888d-4137-89a5-221e5a1bc171/d68b35fd-c62c-4cb2-9479-1cd357042dd9"
-					(reference "C14")
+					(reference "C13")
 					(unit 1)
 				)
@@
 		(dnp no)
 		(fields_autoplaced yes)
-		(property "Reference" "#PWR063"
+		(property "Reference" "#PWR062"
 			(at 187.96 142.24 0)
 			(effects
@@
 			(project "CMPE2750"
 				(path "/a86318a1-888d-4137-89a5-221e5a1bc171/d68b35fd-c62c-4cb2-9479-1cd357042dd9"
-					(reference "#PWR063")
+					(reference "#PWR062")
 					(unit 1)
 				)
@@
 		(on_board yes)
 		(dnp no)
-		(property "Reference" "#PWR060"
+		(property "Reference" "#PWR059"
 			(at 69.85 81.28 0)
 			(effects
@@
 			(project ""
 				(path "/a86318a1-888d-4137-89a5-221e5a1bc171/d68b35fd-c62c-4cb2-9479-1cd357042dd9"
-					(reference "#PWR060")
+					(reference "#PWR059")
 					(unit 1)
 				)
@@
 		(dnp no)
 		(fields_autoplaced yes)
-		(property "Reference" "#PWR065"
+		(property "Reference" "#PWR064"
 			(at 58.42 148.59 0)
 			(effects
@@
 			(project ""
 				(path "/a86318a1-888d-4137-89a5-221e5a1bc171/d68b35fd-c62c-4cb2-9479-1cd357042dd9"
-					(reference "#PWR065")
+					(reference "#PWR064")
 					(unit 1)
 				)
@@
 		(dnp no)
 		(fields_autoplaced yes)
-		(property "Reference" "#PWR053"
+		(property "Reference" "#PWR052"
 			(at 269.24 29.21 0)
 			(effects
@@
 			(project "CMPE2750"
 				(path "/a86318a1-888d-4137-89a5-221e5a1bc171/d68b35fd-c62c-4cb2-9479-1cd357042dd9"
-					(reference "#PWR053")
+					(reference "#PWR052")
 					(unit 1)
 				)

Commit message: Component placing partly done. Saving before overwriting the pcb with the templating script output
Parts:
- J7, J8: value Conn_02x02_Counter_Clockwise -> Conn_02x02_Odd_Even; symbol Connector_Generic:Conn_02x02_Counter_Clockwise -> Connector_Generic:Conn_02x02_Odd_Even
Connections:
- net ADC: now also J7.4 (Pin_4); no longer J7.3 (Pin_3)
- net Ooutput_2b: now also J8.2 (Pin_2); no longer J8.4 (Pin_4)
- net Output_2a: now also J7.2 (Pin_2); no longer J7.4 (Pin_4)
- net in_filter_input: now also J7.3 (Pin_3); no longer J7.2 (Pin_2)
- net out_conditioning: now also J8.4 (Pin_4); no longer J8.3 (Pin_3)
- net out_filt_input: now also J8.3 (Pin_3); no longer J8.2 (Pin_2)
Changed lines of the file:
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@@
 	)
 	(symbol
-		(lib_id "Connector_Generic:Conn_02x02_Counter_Clockwise")
+		(lib_id "Connector_Generic:Conn_02x02_Odd_Even")
 		(at 252.73 62.23 0)
 		(unit 1)
@@
 			)
 		)
-		(property "Value" "Conn_02x02_Counter_Clockwise"
+		(property "Value" "Conn_02x02_Odd_Even"
 			(at 254 58.42 0)
 			(effects
@@
 			)
 		)
-		(property "Description" "Generic connector, double row, 02x02, counter clockwise pin numbering scheme (similar to DIP package numbering), script generated (kicad-library-utils/schlib/autogen/connector/)"
+		(property "Description" "Generic connector, double row, 02x02, odd/even pin numbering scheme (row 1 odd numbers, row 2 even numbers), script generated (kicad-library-utils/schlib/autogen/connector/)"
 			(at 252.73 62.23 0)
 			(effects
@@
 	)
 	(symbol
-		(lib_id "Connector_Generic:Conn_02x02_Counter_Clockwise")
+		(lib_id "Connector_Generic:Conn_02x02_Odd_Even")
 		(at 144.78 99.06 0)
 		(unit 1)
@@
 			)
 		)
-		(property "Value" "Conn_02x02_Counter_Clockwise"
+		(property "Value" "Conn_02x02_Odd_Even"
 			(at 146.05 95.25 0)
 			(effects
@@
 			)
 		)
-		(property "Description" "Generic connector, double row, 02x02, counter clockwise pin numbering scheme (similar to DIP package numbering), script generated (kicad-library-utils/schlib/autogen/connector/)"
+		(property "Description" "Generic connector, double row, 02x02, odd/even pin numbering scheme (row 1 odd numbers, row 2 even numbers), script generated (kicad-library-utils/schlib/autogen/connector/)"
 			(at 144.78 99.06 0)
 			(effects
