File: filters_and_amps.kicad_sch (KiCad schematic)
At the start: 32 parts, among them J7 Conn_02x02_Odd_Even, J8 Conn_02x02_Odd_Even, U4 OPA1678IDR, U5 OPA1678IDR, U6 OPA1678IDR

Commit message: finished
Parts:
- removed C16, C17, C18, C19: 10nF, Capacitor_SMD:C_0805_2012Metric, symbol CMPE2750:GRM2195C1H103FA01D
- removed C20, C22: 680pF, Capacitor_SMD:C_0402_1005Metric, symbol CMPE2750:CC1206FRNPO9BN681
- removed C21, C23: 3.3nF, Capacitor_SMD:C_0603_1608Metric, symbol CMPE2750:1206N332F500CT
- removed R39, R43: 26.7kΩ, Resistor_SMD:R_0603_1608Metric, symbol CMPE2750:0402WGF3832TCE
- removed R40, R41, R44, R45: 15.4kΩ, Resistor_SMD:R_0603_1608Metric, symbol CMPE2750:RT0603BRD0722K1L
- removed R42, R46: 5.49kΩ, Resistor_SMD:R_0402_1005Metric, symbol CMPE2750:RT0402BRD077K87L
- added C16, C17: 100nF, Capacitor_SMD:C_0402_1005Metric, symbol CMPE2750:CL05B104KP5NNNC
- added U13, U14: TLC04CD, D8, symbol CMPE2750:TLC04CD
Connections:
- net -5V: now also C16.2, C17.2, U13.1 (CLKIN), U13.4 (VCC-), U14.1 (CLKIN), U14.4 (VCC-)
- net GND: now also U13.3 (LS), U13.6 (AGND), U14.3 (LS), U14.6 (AGND)
- net VBUS: now also C16.1, C17.1, U13.7 (VCC+), U14.7 (VCC+)
- net in_filter_input: now also U13.8 (FILTERIN)
- net out_filt_input: now also U14.8 (FILTERIN)
- net Ooutput_2b renamed output_filter
- net output_filter: now also U14.5 (FILTEROUT)
- net Output_2a renamed input_filter
- net input_filter: now also U13.5 (FILTEROUT)
- new net CLK_{filt}: U13.2 (CLKR), U14.2 (CLKR)
Other:
- removed sheet filter_amps
