File: switch_leds.kicad_sch (KiCad schematic)
At the start: 65 parts, among them J4 Conn_01x02, Q1 NPN, Q10 NPN, Q11 NPN, Q12 NPN, Q13 NPN, Q14 NPN, Q15 NPN, Q16 NPN, Q2 NPN, Q3 NPN, Q4 NPN, Q5 NPN, Q6 NPN, Q7 NPN, Q8 NPN, Q9 NPN, U49 NSI45015WT1G, U50 NSI45015WT1G, U51 NSI45015WT1G, U52 NSI45015WT1G, U53 NSI45015WT1G, U54 NSI45015WT1G, U55 NSI45015WT1G, U56 NSI45015WT1G, U57 NSI45015WT1G, U58 NSI45015WT1G, U59 NSI45015WT1G, U60 NSI45015WT1G, U61 NSI45015WT1G, U62 NSI45015WT1G, U63 NSI45015WT1G, U64 NSI45015WT1G

Commit message: Finished the display and input switch schematics. Also added input buffers to the inputs and made them differential
Parts:
- Q1, Q10, Q11, Q12, Q13, Q14, Q15, Q16, Q2, Q3, Q4, Q5, Q6, Q7, Q8, Q9: value NPN -> 2N7002; footprint (none) -> Package_TO_SOT_SMD:SOT-23; symbol Simulation_SPICE:NPN -> Transistor_FET:2N7002
- R41, R42, R43, R44, R45, R46, R47, R48, R49, R50, R51, R52, R53, R54, R55, R56: value 22kΩ -> 4.7kΩ; footprint (none) -> Resistor_SMD:R_1206_3216Metric
Connections:
- net GND: now also Q1.2 (S), Q10.2 (S), Q11.2 (S), Q12.2 (S), Q13.2 (S), Q14.2 (S), Q15.2 (S), Q16.2 (S), Q2.2 (S), Q3.2 (S), Q4.2 (S), Q5.2 (S), Q6.2 (S), Q7.2 (S), Q8.2 (S), Q9.2 (S); no longer Q1.3 (E), Q10.3 (E), Q11.3 (E), Q12.3 (E), Q13.3 (E), Q14.3 (E), Q15.3 (E), Q16.3 (E), Q2.3 (E), Q3.3 (E), Q4.3 (E), Q5.3 (E), Q6.3 (E), Q7.3 (E), Q8.3 (E), Q9.3 (E)
- net at R52.2: now also Q12.1 (G); no longer Q12.2 (B)
- net at D16.1 (K): now also Q14.3 (D); no longer Q14.1 (C)
- net at Q13.1 (G): now also R53.2; no longer D15.1 (K)
- net at Q6.1 (G): now also R46.2; no longer D8.1 (K)
- net at R51.2: now also Q11.1 (G); no longer Q11.2 (B)
- net at D14.1 (K): now also Q12.3 (D); no longer Q12.1 (C)
- net at D11.1 (K): now also Q9.3 (D); no longer Q9.1 (C)
- net at Q4.1 (G): now also R44.2; no longer D6.1 (K)
- net at R50.2: now also Q10.1 (G); no longer Q10.2 (B)
- net at D3.1 (K): now also Q1.3 (D); no longer Q1.1 (C)
- net at D5.1 (K): now also Q3.3 (D); no longer Q3.1 (C)
- net at Q8.1 (G): now also R48.2; no longer D10.1 (K)
- net at R45.2: now also Q5.1 (G); no longer Q5.2 (B)
- net at R42.2: now also Q2.1 (G); no longer Q2.2 (B)
- net at D7.1 (K): now also Q5.3 (D); no longer Q5.1 (C)
- net at Q16.1 (G): now also R56.2; no longer D18.1 (K)
- net at D12.1 (K): now also Q10.3 (D); no longer Q10.1 (C)
- net at R49.2: now also Q9.1 (G); no longer Q9.2 (B)
- net at Q7.1 (G): now also R47.2; no longer D9.1 (K)
- net at R43.2: now also Q3.1 (G); no longer Q3.2 (B)
- net at R41.2: now also Q1.1 (G); no longer Q1.2 (B)
- net at R54.2: now also Q14.1 (G); no longer Q14.2 (B)
- net at D13.1 (K): now also Q11.3 (D); no longer Q11.1 (C)
- net at R55.2: now also Q15.1 (G); no longer Q15.2 (B)
- net at D17.1 (K): now also Q15.3 (D); no longer Q15.1 (C)
- net at D4.1 (K): now also Q2.3 (D); no longer Q2.1 (C)
- new net: D15.1 (K), Q13.3 (D)
- new net: D8.1 (K), Q6.3 (D)
- new net: D6.1 (K), Q4.3 (D)
- new net: D10.1 (K), Q8.3 (D)
- new net: D18.1 (K), Q16.3 (D)
- new net: D9.1 (K), Q7.3 (D)

Commit message: Schematic is done?
Parts:
- J4: footprint (none) -> Connector_PinHeader_2.54mm:PinHeader_1x02_P2.54mm_Vertical
Changed lines of the file:
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@@
 			)
 		)
-		(property "Footprint" ""
+		(property "Footprint" "Connector_PinHeader_2.54mm:PinHeader_1x02_P2.54mm_Vertical"
 			(at 29.21 24.13 0)
 			(effects

Commit message: Swapped the current limiting diodes for resistors. They *should* be good enough under normal operating conditions. Also added some pull-down resistors. Done?
Parts:
- removed U49, U50, U51, U52, U53, U54, U55, U56, U57, U58, U59, U60, U61, U62, U63, U64: NSI45015WT1G, SOD123-2_ONS, symbol CMPE2750:NSI45015WT1G
- added R175, R176, R177, R178, R179, R180, R181, R182, R183, R184, R185, R186, R187, R188, R189, R190: 133Ω, Resistor_SMD:R_0603_1608Metric, symbol CMPE2750:RT0603BRD07133RL
Connections:
- net sl_power: now also R175.2, R176.2, R177.2, R178.2, R179.2, R180.2, R181.2, R182.2, R183.2, R184.2, R185.2, R186.2, R187.2, R188.2, R189.2, R190.2
- net at D9.2 (A): now also R182.1
- net at D4.2 (A): now also R176.1
- net at D16.2 (A): now also R185.1
- net at D10.2 (A): now also R179.1
- net at D14.2 (A): now also R180.1
- net at D11.2 (A): now also R189.1
- net at D8.2 (A): now also R187.1
- net at D3.2 (A): now also R175.1
- net at D5.2 (A): now also R177.1
- net at D6.2 (A): now also R178.1
- net at D15.2 (A): now also R190.1
- net at D7.2 (A): now also R188.1
- net at D18.2 (A): now also R181.1
- net at D13.2 (A): now also R183.1
- net at D17.2 (A): now also R184.1
- net at D12.2 (A): now also R186.1

Commit message: Added mounting holes to the schematic, reset the annotations, updated a few footprints, and fixed some issues that were discovered on the ERC.
Parts:
- renumbered D7 to D10, D13 to D11, D14 to D13, D11 to D14, D9 to D7, D10 to D9, J4 to J10, Q1 to Q51, Q2 to Q52, Q3 to Q53, Q4 to Q54, Q7 to Q55, Q6 to Q56, Q8 to Q57, Q5 to Q58, Q11 to Q59, Q10 to Q60, Q12 to Q61, Q9 to Q62, Q13 to Q63, Q14 to Q64, Q15 to Q65, Q16 to Q66, R175 to R159, R176 to R160, R177 to R161, R178 to R162, R41 to R163, R42 to R164, R43 to R165, R44 to R166, R182 to R167, R187 to R168, R179 to R169, R188 to R170, R47 to R171, R46 to R172, R48 to R173, R45 to R174, R183 to R175, R186 to R176, R180 to R177, R189 to R178, R51 to R179, R50 to R180, R52 to R181, R49 to R182, R190 to R183, R185 to R184, R184 to R185, R181 to R186, R53 to R187, R54 to R188, R55 to R189, R56 to R190

Commit message: Component placing partly done. Saving before overwriting the pcb with the templating script output
Parts:
- R163, R164, R165, R166, R171, R172, R173, R174, R179, R180, R181, R182, R187, R188, R189, R190: footprint Resistor_SMD:R_1206_3216Metric -> Resistor_SMD:R_0402_1005Metric; symbol Device:R_US -> CMPE2750:AC0402FR-074K7L
